Commit message: Change mesh paths to asset folder

File: sample_description/urdf/low_cost_robot.urdf (robot description, URDF)
Before this commit: robot low_cost_robot, 7 links, 6 joints
Links:
- link base_link: geometry collision mesh filename=meshes/base_link.stl scale=0.001 0.001 0.001; visual mesh filename=meshes/base_link.stl scale=0.001 0.001 0.001
- link gripper_moving_1: geometry collision mesh filename=meshes/gripper_moving_1.stl scale=0.001 0.001 0.001; visual mesh filename=meshes/gripper_moving_1.stl scale=0.001 0.001 0.001
- link gripper_static_1: geometry collision mesh filename=meshes/gripper_static_1.stl scale=0.001 0.001 0.001; visual mesh filename=meshes/gripper_static_1.stl scale=0.001 0.001 0.001
- link link1_1: geometry collision mesh filename=meshes/link1_1.stl scale=0.001 0.001 0.001; visual mesh filename=meshes/link1_1.stl scale=0.001 0.001 0.001
- link link2_1: geometry collision mesh filename=meshes/link2_1.stl scale=0.001 0.001 0.001; visual mesh filename=meshes/link2_1.stl scale=0.001 0.001 0.001
- link link3_1: geometry collision mesh filename=meshes/link3_1.stl scale=0.001 0.001 0.001; visual mesh filename=meshes/link3_1.stl scale=0.001 0.001 0.001
- link link4_1: geometry collision mesh filename=meshes/link4_1.stl scale=0.001 0.001 0.001; visual mesh filename=meshes/link4_1.stl scale=0.001 0.001 0.001
